File: BusBoard/BusBoard.kicad_pcb (KiCad board)
At the start: 2 copper layers, 340 x 50 mm, 45 parts, among them J1 Conn_L10, J10 Conn_L1, J11 Conn_R1, J12 Conn_R2, J13 Conn_R3, J14 Conn_R4, J15 Conn_R5, J16 Conn_R6, J17 Conn_R7, J18 Conn_R8, J19 Conn_R9, J2 Conn_L9, J20 Conn_R10, J21 From Supply, J22 To Busboard, J3 Conn_L8, J4 Conn_L7, J5 Conn_L6, J6 Conn_L5, J7 Conn_L4, J8 Conn_L3, J9 Conn_L2

Commit message: fix 16pin layout
Parts:
- removed LED1: Red, LED_THT:LED_D3.0mm
- removed LED2: Green, LED_THT:LED_D3.0mm
- removed LED3: Blue, LED_THT:LED_D3.0mm
- added D1: LED_Red, LED_THT:LED_D3.0mm, F.Cu at (195.5, 149.5)
- added D2: LED_Grean, LED_THT:LED_D3.0mm, F.Cu at (213.6, 149.6)
- added D3: LED_Blue, LED_THT:LED_D3.0mm, F.Cu at (233.9, 149.6)
- moved J22 1.99 mm to (196.3, 160.3)
- moved J14 1.73 mm to (284.3, 137.0)
- moved J17 1.73 mm to (326.5, 137.0)
- moved C2 1.73 mm to (189.9, 141.7)
- moved C3 1.73 mm to (189.9, 149.5)
- moved C4 1.73 mm to (206.7, 136.2)
- moved C5 1.73 mm to (207.9, 141.8)
- moved C6 1.73 mm to (207.9, 149.6)
- moved C8 1.73 mm to (226.1, 141.8)
- moved C9 1.73 mm to (226.1, 149.6)
- moved J10 1.73 mm to (174.8, 137.0)
- moved J21 1.73 mm to (221.5, 127.1)
- moved J3 1.73 mm to (76.1, 137.0)
- moved J6 1.73 mm to (118.4, 137.0)
- moved J7 1.73 mm to (132.5, 137.0)
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Connections:
- J1 pad 1: GATE -> -12V
- J1 pad 10: GND -> +12V
- J1 pad 11: GND -> +5V
- J1 pad 12: GND -> +5V
- J1 pad 13: GND -> CV
- J1 pad 14: GND -> CV
- J1 pad 15: -12V -> GATE
- J1 pad 16: -12V -> GATE
- J1 pad 2: GATE -> -12V
- J1 pad 3: CV -> GND
- J1 pad 4: CV -> GND
- J1 pad 5: +5V -> GND
- J1 pad 6: +5V -> GND
- J1 pad 7: +12V -> GND
- J1 pad 8: +12V -> GND
- J1 pad 9: GND -> +12V
- J10 pad 1: GATE -> -12V
- J10 pad 10: GND -> +12V
- J10 pad 11: GND -> +5V
- J10 pad 12: GND -> +5V
- J10 pad 13: GND -> CV
- J10 pad 14: GND -> CV
- J10 pad 15: -12V -> GATE
- J10 pad 16: -12V -> GATE
- J10 pad 2: GATE -> -12V
- J10 pad 3: CV -> GND
- J10 pad 4: CV -> GND
- J10 pad 5: +5V -> GND
- J10 pad 6: +5V -> GND
- J10 pad 7: +12V -> GND
- J10 pad 8: +12V -> GND
- J10 pad 9: GND -> +12V
- J11 pad 1: GATE -> -12V
- J11 pad 10: GND -> +12V
- J11 pad 11: GND -> +5V
- J11 pad 12: GND -> +5V
- J11 pad 13: GND -> CV
- J11 pad 14: GND -> CV
- J11 pad 15: -12V -> GATE
- J11 pad 16: -12V -> GATE
- J11 pad 2: GATE -> -12V
- J11 pad 3: CV -> GND
- J11 pad 4: CV -> GND
- J11 pad 5: +5V -> GND
- J11 pad 6: +5V -> GND
- J11 pad 7: +12V -> GND
- J11 pad 8: +12V -> GND
- J11 pad 9: GND -> +12V
- J12 pad 1: GATE -> -12V
- J12 pad 10: GND -> +12V
- J12 pad 11: GND -> +5V
- J12 pad 12: GND -> +5V
- J12 pad 13: GND -> CV
- J12 pad 14: GND -> CV
- J12 pad 15: -12V -> GATE
- J12 pad 16: -12V -> GATE
- J12 pad 2: GATE -> -12V
- J12 pad 3: CV -> GND
- J12 pad 4: CV -> GND
- J12 pad 5: +5V -> GND
- J12 pad 6: +5V -> GND
- J12 pad 7: +12V -> GND
- J12 pad 8: +12V -> GND
- J12 pad 9: GND -> +12V
- J13 pad 1: GATE -> -12V
- J13 pad 10: GND -> +12V
- J13 pad 11: GND -> +5V
- J13 pad 12: GND -> +5V
- J13 pad 13: GND -> CV
- J13 pad 14: GND -> CV
- J13 pad 15: -12V -> GATE
- J13 pad 16: -12V -> GATE
- J13 pad 2: GATE -> -12V
- J13 pad 3: CV -> GND
- J13 pad 4: CV -> GND
- J13 pad 5: +5V -> GND
- J13 pad 6: +5V -> GND
- J13 pad 7: +12V -> GND
- J13 pad 8: +12V -> GND
- J13 pad 9: GND -> +12V
- J14 pad 1: GATE -> -12V
- J14 pad 10: GND -> +12V
- J14 pad 11: GND -> +5V
- J14 pad 12: GND -> +5V
- J14 pad 13: GND -> CV
- J14 pad 14: GND -> CV
- J14 pad 15: -12V -> GATE
- J14 pad 16: -12V -> GATE
- J14 pad 2: GATE -> -12V
- J14 pad 3: CV -> GND
- J14 pad 4: CV -> GND
- J14 pad 5: +5V -> GND
- J14 pad 6: +5V -> GND
- J14 pad 7: +12V -> GND
- J14 pad 8: +12V -> GND
- J14 pad 9: GND -> +12V
- J15 pad 1: GATE -> -12V
- J15 pad 10: GND -> +12V
- J15 pad 11: GND -> +5V
- J15 pad 12: GND -> +5V
- J15 pad 13: GND -> CV
- J15 pad 14: GND -> CV
- J15 pad 15: -12V -> GATE
- J15 pad 16: -12V -> GATE
- J15 pad 2: GATE -> -12V
- J15 pad 3: CV -> GND
- J15 pad 4: CV -> GND
- J15 pad 5: +5V -> GND
- J15 pad 6: +5V -> GND
- J15 pad 7: +12V -> GND
- J15 pad 8: +12V -> GND
- J15 pad 9: GND -> +12V
- J16 pad 1: GATE -> -12V
- J16 pad 10: GND -> +12V
- J16 pad 11: GND -> +5V
- J16 pad 12: GND -> +5V
- J16 pad 13: GND -> CV
- J16 pad 14: GND -> CV
- J16 pad 15: -12V -> GATE
- J16 pad 16: -12V -> GATE
- J16 pad 2: GATE -> -12V
- J16 pad 3: CV -> GND
- J16 pad 4: CV -> GND
- J16 pad 5: +5V -> GND
- J16 pad 6: +5V -> GND
- J16 pad 7: +12V -> GND
- J16 pad 8: +12V -> GND
- J16 pad 9: GND -> +12V
- J17 pad 1: GATE -> -12V
- J17 pad 10: GND -> +12V
- J17 pad 11: GND -> +5V
- J17 pad 12: GND -> +5V
- J17 pad 13: GND -> CV
- J17 pad 14: GND -> CV
- J17 pad 15: -12V -> GATE
- J17 pad 16: -12V -> GATE
- J17 pad 2: GATE -> -12V
- J17 pad 3: CV -> GND
- J17 pad 4: CV -> GND
- J17 pad 5: +5V -> GND
- J17 pad 6: +5V -> GND
- J17 pad 7: +12V -> GND
- J17 pad 8: +12V -> GND
- J17 pad 9: GND -> +12V
- J18 pad 1: GATE -> -12V
- J18 pad 10: GND -> +12V
- J18 pad 11: GND -> +5V
- J18 pad 12: GND -> +5V
- J18 pad 13: GND -> CV
- J18 pad 14: GND -> CV
- J18 pad 15: -12V -> GATE
- J18 pad 16: -12V -> GATE
- J18 pad 2: GATE -> -12V
- J18 pad 3: CV -> GND
- J18 pad 4: CV -> GND
- J18 pad 5: +5V -> GND
- J18 pad 6: +5V -> GND
- J18 pad 7: +12V -> GND
- J18 pad 8: +12V -> GND
- J18 pad 9: GND -> +12V
- J19 pad 1: GATE -> -12V
- J19 pad 10: GND -> +12V
- J19 pad 11: GND -> +5V
- J19 pad 12: GND -> +5V
- J19 pad 13: GND -> CV
- J19 pad 14: GND -> CV
- J19 pad 15: -12V -> GATE
- J19 pad 16: -12V -> GATE
- J19 pad 2: GATE -> -12V
- J19 pad 3: CV -> GND
- J19 pad 4: CV -> GND
- J19 pad 5: +5V -> GND
- J19 pad 6: +5V -> GND
- J19 pad 7: +12V -> GND
- J19 pad 8: +12V -> GND
- J19 pad 9: GND -> +12V
- J2 pad 1: GATE -> -12V
- J2 pad 10: GND -> +12V
- J2 pad 11: GND -> +5V
- J2 pad 12: GND -> +5V
- J2 pad 13: GND -> CV
- J2 pad 14: GND -> CV
- J2 pad 15: -12V -> GATE
- J2 pad 16: -12V -> GATE
- J2 pad 2: GATE -> -12V
- J2 pad 3: CV -> GND
- J2 pad 4: CV -> GND
- J2 pad 5: +5V -> GND
- J2 pad 6: +5V -> GND
- J2 pad 7: +12V -> GND
- J2 pad 8: +12V -> GND
- J2 pad 9: GND -> +12V
- J20 pad 1: GATE -> -12V
- J20 pad 10: GND -> +12V
- J20 pad 11: GND -> +5V
- J20 pad 12: GND -> +5V
- J20 pad 13: GND -> CV
- J20 pad 14: GND -> CV
- J20 pad 15: -12V -> GATE
- J20 pad 16: -12V -> GATE
- J20 pad 2: GATE -> -12V
- J20 pad 3: CV -> GND
- J20 pad 4: CV -> GND
- J20 pad 5: +5V -> GND
- J20 pad 6: +5V -> GND
- J20 pad 7: +12V -> GND
- J20 pad 8: +12V -> GND
- J20 pad 9: GND -> +12V
- J3 pad 1: GATE -> -12V
- J3 pad 10: GND -> +12V
- J3 pad 11: GND -> +5V
- J3 pad 12: GND -> +5V
- J3 pad 13: GND -> CV
- J3 pad 14: GND -> CV
- J3 pad 15: -12V -> GATE
- J3 pad 16: -12V -> GATE
- J3 pad 2: GATE -> -12V
- J3 pad 3: CV -> GND
- J3 pad 4: CV -> GND
- J3 pad 5: +5V -> GND
- J3 pad 6: +5V -> GND
- J3 pad 7: +12V -> GND
- J3 pad 8: +12V -> GND
- J3 pad 9: GND -> +12V
- J4 pad 1: GATE -> -12V
- J4 pad 10: GND -> +12V
- J4 pad 11: GND -> +5V
- J4 pad 12: GND -> +5V
- J4 pad 13: GND -> CV
- J4 pad 14: GND -> CV
- J4 pad 15: -12V -> GATE
- J4 pad 16: -12V -> GATE
- J4 pad 2: GATE -> -12V
- J4 pad 3: CV -> GND
- J4 pad 4: CV -> GND
- J4 pad 5: +5V -> GND
- J4 pad 6: +5V -> GND
- J4 pad 7: +12V -> GND
- J4 pad 8: +12V -> GND
- J4 pad 9: GND -> +12V
- J5 pad 1: GATE -> -12V
- J5 pad 10: GND -> +12V
- J5 pad 11: GND -> +5V
- J5 pad 12: GND -> +5V
- J5 pad 13: GND -> CV
- J5 pad 14: GND -> CV
- J5 pad 15: -12V -> GATE
- J5 pad 16: -12V -> GATE
- J5 pad 2: GATE -> -12V
- J5 pad 3: CV -> GND
- J5 pad 4: CV -> GND
- J5 pad 5: +5V -> GND
- J5 pad 6: +5V -> GND
- J5 pad 7: +12V -> GND
- J5 pad 8: +12V -> GND
- J5 pad 9: GND -> +12V
- J6 pad 1: GATE -> -12V
- J6 pad 10: GND -> +12V
- J6 pad 11: GND -> +5V
- J6 pad 12: GND -> +5V
- J6 pad 13: GND -> CV
- J6 pad 14: GND -> CV
- J6 pad 15: -12V -> GATE
- J6 pad 16: -12V -> GATE
- J6 pad 2: GATE -> -12V
- J6 pad 3: CV -> GND
- J6 pad 4: CV -> GND
- J6 pad 5: +5V -> GND
- J6 pad 6: +5V -> GND
- J6 pad 7: +12V -> GND
- J6 pad 8: +12V -> GND
- J6 pad 9: GND -> +12V
- J7 pad 1: GATE -> -12V
- J7 pad 10: GND -> +12V
- J7 pad 11: GND -> +5V
- J7 pad 12: GND -> +5V
- J7 pad 13: GND -> CV
- J7 pad 14: GND -> CV
- J7 pad 15: -12V -> GATE
- J7 pad 16: -12V -> GATE
- J7 pad 2: GATE -> -12V
- J7 pad 3: CV -> GND
- J7 pad 4: CV -> GND
- J7 pad 5: +5V -> GND
- J7 pad 6: +5V -> GND
- J7 pad 7: +12V -> GND
- J7 pad 8: +12V -> GND
- J7 pad 9: GND -> +12V
- J8 pad 1: GATE -> -12V
- J8 pad 10: GND -> +12V
- J8 pad 11: GND -> +5V
- J8 pad 12: GND -> +5V
- J8 pad 13: GND -> CV
- J8 pad 14: GND -> CV
- J8 pad 15: -12V -> GATE
- J8 pad 16: -12V -> GATE
- J8 pad 2: GATE -> -12V
- J8 pad 3: CV -> GND
- J8 pad 4: CV -> GND
- J8 pad 5: +5V -> GND
- J8 pad 6: +5V -> GND
- J8 pad 7: +12V -> GND
- J8 pad 8: +12V -> GND
- J8 pad 9: GND -> +12V
- J9 pad 1: GATE -> -12V
- J9 pad 10: GND -> +12V
- J9 pad 11: GND -> +5V
- J9 pad 12: GND -> +5V
- J9 pad 13: GND -> CV
- J9 pad 14: GND -> CV
- J9 pad 15: -12V -> GATE
- J9 pad 16: -12V -> GATE
- J9 pad 2: GATE -> -12V
- J9 pad 3: CV -> GND
- J9 pad 4: CV -> GND
- J9 pad 5: +5V -> GND
- J9 pad 6: +5V -> GND
- J9 pad 7: +12V -> GND
- J9 pad 8: +12V -> GND
- J9 pad 9: GND -> +12V
Routing:
- net -12V: track 378.1 -> 395.2 mm, vias 7 -> 5
- net +5V: track 390.6 -> 380.3 mm, vias 7 -> 5
- net CV: track 358.3 -> 361.8 mm, vias 1 -> 0
- net +12V: track 413.9 -> 416.8 mm, vias 14 -> 5
- net GATE: track 367.0 -> 368.0 mm, vias 3 -> 4
Other:
- board text added: "GATE"
