File: PSU/PSU.kicad_pcb (KiCad board)
At the start: 2 copper layers, 90 x 160 mm, 31 parts, among them J1 From Supply, J2 To Busboard, J3 To Dummy Load

Commit message: Remove generated KiCad files
Connections:
- J2 pad 1: Net-(C11-Pad2) -> Net-(C18-Pad1)
- J2 pad 2: GND -> Net-(C4-Pad1)
- J2 pad 3: Net-(C4-Pad1) -> GND
- J2 pad 4: Net-(C18-Pad1) -> Net-(C11-Pad2)
Routing:
- net Net-(C18-Pad1): track 96.2 -> 115.2 mm
- net Net-(C11-Pad2): track 76.9 -> 79.0 mm
