File: SSI2130_VCO/SSI2130_VCO_Power-VREF.kicad_sch (KiCad schematic)
At the start: 14 parts, among them IC1 LM4040AELT-2.5, J1 Conn_02x08_Odd_Even, U1 TLV9062IDR

Commit message: add TZ circuit
Connections:
- net +5V_IN renamed +5V
